File: RNA.sch (KiCad schematic (older format))
At the start: 71 parts

Commit message: add connectors
Parts:
- removed U?: STM32F303C6Tx, Package_QFP:LQFP-48_7x7mm_P0.5mm, symbol MCU_ST_STM32F3:STM32F303C6Tx
- added J?: USB_C_Receptacle_USB2.0, symbol Connector:USB_C_Receptacle_USB2.0
- added J?: Conn_01x06, symbol Connector_Generic:Conn_01x06
- added J?: AudioJack4, symbol Connector:AudioJack4
- added R?: 1.5k, symbol Device:R_Small
- added U?: USBLC6-2SC6, Package_TO_SOT_SMD:SOT-23-6, symbol Power_Protection:USBLC6-2SC6
- added U?: STM32F302CBTx, Package_QFP:LQFP-48_7x7mm_P0.5mm, symbol MCU_ST_STM32F3:STM32F302CBTx
Connections:
- net labels added: NRST, OSC_IN, OSC_OUT, SWCLK, SWDIO, SWO, VBUS
- wire segments 208 -> 252

Commit message: add footprint
Parts:
- SW? (x32): footprint (none) -> keyswitch:PG1350_socket
Changed lines of the file:
@@
 F 0 "SW?" H 6400 3178 50  0000 C CNN
 F 1 "SW_Push_45deg" H 6400 3087 50  0000 C CNN
-F 2 "" H 6400 2900 50  0001 C CNN
+F 2 "keyswitch:PG1350_socket" H 6400 2900 50  0001 C CNN
 F 3 "" H 6400 2900 50  0001 C CNN
 	1    6400 2900
@@
 F 0 "SW?" H 7050 3178 50  0000 C CNN
 F 1 "SW_Push_45deg" H 7050 3087 50  0000 C CNN
-F 2 "" H 7050 2900 50  0001 C CNN
+F 2 "keyswitch:PG1350_socket" H 7050 2900 50  0001 C CNN
 F 3 "" H 7050 2900 50  0001 C CNN
 	1    7050 2900
@@
 F 0 "SW?" H 7700 3178 50  0000 C CNN
 F 1 "SW_Push_45deg" H 7700 3087 50  0000 C CNN
-F 2 "" H 7700 2900 50  0001 C CNN
+F 2 "keyswitch:PG1350_socket" H 7700 2900 50  0001 C CNN
 F 3 "" H 7700 2900 50  0001 C CNN
 	1    7700 2900
@@
 F 0 "SW?" H 8350 3178 50  0000 C CNN
 F 1 "SW_Push_45deg" H 8350 3087 50  0000 C CNN
-F 2 "" H 8350 2900 50  0001 C CNN
+F 2 "keyswitch:PG1350_socket" H 8350 2900 50  0001 C CNN
 F 3 "" H 8350 2900 50  0001 C CNN
 	1    8350 2900
@@
 F 0 "SW?" H 9000 3178 50  0000 C CNN
 F 1 "SW_Push_45deg" H 9000 3087 50  0000 C CNN
-F 2 "" H 9000 2900 50  0001 C CNN
+F 2 "keyswitch:PG1350_socket" H 9000 2900 50  0001 C CNN
 F 3 "" H 9000 2900 50  0001 C CNN
 	1    9000 2900
@@
 F 0 "SW?" H 9650 3178 50  0000 C CNN
 F 1 "SW_Push_45deg" H 9650 3087 50  0000 C CNN
-F 2 "" H 9650 2900 50  0001 C CNN
+F 2 "keyswitch:PG1350_socket" H 9650 2900 50  0001 C CNN
 F 3 "" H 9650 2900 50  0001 C CNN
 	1    9650 2900
@@
 F 0 "SW?" H 6400 3828 50  0000 C CNN
 F 1 "SW_Push_45deg" H 6400 3737 50  0000 C CNN
-F 2 "" H 6400 3550 50  0001 C CNN
+F 2 "keyswitch:PG1350_socket" H 6400 3550 50  0001 C CNN
 F 3 "" H 6400 3550 50  0001 C CNN
 	1    6400 3550
@@
 F 0 "SW?" H 7050 3828 50  0000 C CNN
 F 1 "SW_Push_45deg" H 7050 3737 50  0000 C CNN
-F 2 "" H 7050 3550 50  0001 C CNN
+F 2 "keyswitch:PG1350_socket" H 7050 3550 50  0001 C CNN
 F 3 "" H 7050 3550 50  0001 C CNN
 	1    7050 3550
@@
 F 0 "SW?" H 7700 3828 50  0000 C CNN
 F 1 "SW_Push_45deg" H 7700 3737 50  0000 C CNN
-F 2 "" H 7700 3550 50  0001 C CNN
+F 2 "keyswitch:PG1350_socket" H 7700 3550 50  0001 C CNN
 F 3 "" H 7700 3550 50  0001 C CNN
 	1    7700 3550
@@
 F 0 "SW?" H 8350 3828 50  0000 C CNN
 F 1 "SW_Push_45deg" H 8350 3737 50  0000 C CNN
-F 2 "" H 8350 3550 50  0001 C CNN
+F 2 "keyswitch:PG1350_socket" H 8350 3550 50  0001 C CNN
 F 3 "" H 8350 3550 50  0001 C CNN
 	1    8350 3550
@@
 F 0 "SW?" H 9000 3828 50  0000 C CNN
 F 1 "SW_Push_45deg" H 9000 3737 50  0000 C CNN
-F 2 "" H 9000 3550 50  0001 C CNN
+F 2 "keyswitch:PG1350_socket" H 9000 3550 50  0001 C CNN
 F 3 "" H 9000 3550 50  0001 C CNN
 	1    9000 3550
@@
 F 0 "SW?" H 9650 3828 50  0000 C CNN
 F 1 "SW_Push_45deg" H 9650 3737 50  0000 C CNN
-F 2 "" H 9650 3550 50  0001 C CNN
+F 2 "keyswitch:PG1350_socket" H 9650 3550 50  0001 C CNN
 F 3 "" H 9650 3550 50  0001 C CNN
 	1    9650 3550
@@
 F 0 "SW?" H 6400 4478 50  0000 C CNN
 F 1 "SW_Push_45deg" H 6400 4387 50  0000 C CNN
-F 2 "" H 6400 4200 50  0001 C CNN
+F 2 "keyswitch:PG1350_socket" H 6400 4200 50  0001 C CNN
 F 3 "" H 6400 4200 50  0001 C CNN
 	1    6400 4200
@@
 F 0 "SW?" H 7050 4478 50  0000 C CNN
 F 1 "SW_Push_45deg" H 7050 4387 50  0000 C CNN
-F 2 "" H 7050 4200 50  0001 C CNN
+F 2 "keyswitch:PG1350_socket" H 7050 4200 50  0001 C CNN
 F 3 "" H 7050 4200 50  0001 C CNN
 	1    7050 4200
@@
 F 0 "SW?" H 7700 4478 50  0000 C CNN
 F 1 "SW_Push_45deg" H 7700 4387 50  0000 C CNN
-F 2 "" H 7700 4200 50  0001 C CNN
+F 2 "keyswitch:PG1350_socket" H 7700 4200 50  0001 C CNN
 F 3 "" H 7700 4200 50  0001 C CNN
 	1    7700 4200
@@
 F 0 "SW?" H 8350 4478 50  0000 C CNN
 F 1 "SW_Push_45deg" H 8350 4387 50  0000 C CNN
-F 2 "" H 8350 4200 50  0001 C CNN
+F 2 "keyswitch:PG1350_socket" H 8350 4200 50  0001 C CNN
 F 3 "" H 8350 4200 50  0001 C CNN
 	1    8350 4200
@@
 F 0 "SW?" H 9000 4478 50  0000 C CNN
 F 1 "SW_Push_45deg" H 9000 4387 50  0000 C CNN
-F 2 "" H 9000 4200 50  0001 C CNN
+F 2 "keyswitch:PG1350_socket" H 9000 4200 50  0001 C CNN
 F 3 "" H 9000 4200 50  0001 C CNN
 	1    9000 4200
@@
 F 0 "SW?" H 9650 4478 50  0000 C CNN
 F 1 "SW_Push_45deg" H 9650 4387 50  0000 C CNN
-F 2 "" H 9650 4200 50  0001 C CNN
+F 2 "keyswitch:PG1350_socket" H 9650 4200 50  0001 C CNN
 F 3 "" H 9650 4200 50  0001 C CNN
 	1    9650 4200
@@
 F 0 "SW?" H 6400 5128 50  0000 C CNN
 F 1 "SW_Push_45deg" H 6400 5037 50  0000 C CNN
-F 2 "" H 6400 4850 50  0001 C CNN
+F 2 "keyswitch:PG1350_socket" H 6400 4850 50  0001 C CNN
 F 3 "" H 6400 4850 50  0001 C CNN
 	1    6400 4850
@@
 F 0 "SW?" H 7050 5128 50  0000 C CNN
 F 1 "SW_Push_45deg" H 7050 5037 50  0000 C CNN
-F 2 "" H 7050 4850 50  0001 C CNN
+F 2 "keyswitch:PG1350_socket" H 7050 4850 50  0001 C CNN
 F 3 "" H 7050 4850 50  0001 C CNN
 	1    7050 4850
@@
 F 0 "SW?" H 7700 5128 50  0000 C CNN
 F 1 "SW_Push_45deg" H 7700 5037 50  0000 C CNN
-F 2 "" H 7700 4850 50  0001 C CNN
+F 2 "keyswitch:PG1350_socket" H 7700 4850 50  0001 C CNN
 F 3 "" H 7700 4850 50  0001 C CNN
 	1    7700 4850
@@
 F 0 "SW?" H 8350 5128 50  0000 C CNN
 F 1 "SW_Push_45deg" H 8350 5037 50  0000 C CNN
-F 2 "" H 8350 4850 50  0001 C CNN
+F 2 "keyswitch:PG1350_socket" H 8350 4850 50  0001 C CNN
 F 3 "" H 8350 4850 50  0001 C CNN
 	1    8350 4850
@@
 F 0 "SW?" H 9000 5128 50  0000 C CNN
 F 1 "SW_Push_45deg" H 9000 5037 50  0000 C CNN
-F 2 "" H 9000 4850 50  0001 C CNN
+F 2 "keyswitch:PG1350_socket" H 9000 4850 50  0001 C CNN
 F 3 "" H 9000 4850 50  0001 C CNN
 	1    9000 4850
@@
 F 0 "SW?" H 9650 5128 50  0000 C CNN
 F 1 "SW_Push_45deg" H 9650 5037 50  0000 C CNN
-F 2 "" H 9650 4850 50  0001 C CNN
+F 2 "keyswitch:PG1350_socket" H 9650 4850 50  0001 C CNN
 F 3 "" H 9650 4850 50  0001 C CNN
 	1    9650 4850
@@
 F 0 "SW?" H 6400 5778 50  0000 C CNN
 F 1 "SW_Push_45deg" H 6400 5687 50  0000 C CNN
-F 2 "" H 6400 5500 50  0001 C CNN
+F 2 "keyswitch:PG1350_socket" H 6400 5500 50  0001 C CNN
 F 3 "" H 6400 5500 50  0001 C CNN
 	1    6400 5500
@@
 F 0 "SW?" H 7050 5778 50  0000 C CNN
 F 1 "SW_Push_45deg" H 7050 5687 50  0000 C CNN
-F 2 "" H 7050 5500 50  0001 C CNN
+F 2 "keyswitch:PG1350_socket" H 7050 5500 50  0001 C CNN
 F 3 "" H 7050 5500 50  0001 C CNN
 	1    7050 5500
@@
 F 0 "SW?" H 7700 5778 50  0000 C CNN
 F 1 "SW_Push_45deg" H 7700 5687 50  0000 C CNN
-F 2 "" H 7700 5500 50  0001 C CNN
+F 2 "keyswitch:PG1350_socket" H 7700 5500 50  0001 C CNN
 F 3 "" H 7700 5500 50  0001 C CNN
 	1    7700 5500
@@
 F 0 "SW?" H 8350 5778 50  0000 C CNN
 F 1 "SW_Push_45deg" H 8350 5687 50  0000 C CNN
-F 2 "" H 8350 5500 50  0001 C CNN
+F 2 "keyswitch:PG1350_socket" H 8350 5500 50  0001 C CNN
 F 3 "" H 8350 5500 50  0001 C CNN
 	1    8350 5500
@@
 F 0 "SW?" H 9000 5778 50  0000 C CNN
 F 1 "SW_Push_45deg" H 9000 5687 50  0000 C CNN
-F 2 "" H 9000 5500 50  0001 C CNN
+F 2 "keyswitch:PG1350_socket" H 9000 5500 50  0001 C CNN
 F 3 "" H 9000 5500 50  0001 C CNN
 	1    9000 5500
@@
 F 0 "SW?" H 9650 5778 50  0000 C CNN
 F 1 "SW_Push_45deg" H 9650 5687 50  0000 C CNN
-F 2 "" H 9650 5500 50  0001 C CNN
+F 2 "keyswitch:PG1350_socket" H 9650 5500 50  0001 C CNN
 F 3 "" H 9650 5500 50  0001 C CNN
 	1    9650 5500
@@
 F 0 "SW?" H 10300 5128 50  0000 C CNN
 F 1 "SW_Push_45deg" H 10300 5037 50  0000 C CNN
-F 2 "" H 10300 4850 50  0001 C CNN
+F 2 "keyswitch:PG1350_socket" H 10300 4850 50  0001 C CNN
 F 3 "" H 10300 4850 50  0001 C CNN
 	1    10300 4850
@@
 F 0 "SW?" H 10300 5778 50  0000 C CNN
 F 1 "SW_Push_45deg" H 10300 5687 50  0000 C CNN
-F 2 "" H 10300 5500 50  0001 C CNN
+F 2 "keyswitch:PG1350_socket" H 10300 5500 50  0001 C CNN
 F 3 "" H 10300 5500 50  0001 C CNN
 	1    10300 5500

Commit message: add more footprint
Parts:
- D? (x32): footprint (none) -> Diode_SMD:D_SOD-123
- J?: footprint (none) -> Connector_PinSocket_2.54mm:PinSocket_1x06_P2.54mm_Vertical
Changed lines of the file:
@@
 F 0 "D?" V 6596 3032 50  0000 R CNN
 F 1 "D_Small" V 6505 3032 50  0000 R CNN
-F 2 "" V 6550 3100 50  0001 C CNN
+F 2 "Diode_SMD:D_SOD-123" V 6550 3100 50  0001 C CNN
 F 3 "~" V 6550 3100 50  0001 C CNN
 	1    6550 3100
@@
 F 0 "D?" V 7246 3032 50  0000 R CNN
 F 1 "D_Small" V 7155 3032 50  0000 R CNN
-F 2 "" V 7200 3100 50  0001 C CNN
+F 2 "Diode_SMD:D_SOD-123" V 7200 3100 50  0001 C CNN
 F 3 "~" V 7200 3100 50  0001 C CNN
 	1    7200 3100
@@
 F 0 "D?" V 7896 3032 50  0000 R CNN
 F 1 "D_Small" V 7805 3032 50  0000 R CNN
-F 2 "" V 7850 3100 50  0001 C CNN
+F 2 "Diode_SMD:D_SOD-123" V 7850 3100 50  0001 C CNN
 F 3 "~" V 7850 3100 50  0001 C CNN
 	1    7850 3100
@@
 F 0 "D?" V 8546 3032 50  0000 R CNN
 F 1 "D_Small" V 8455 3032 50  0000 R CNN
-F 2 "" V 8500 3100 50  0001 C CNN
+F 2 "Diode_SMD:D_SOD-123" V 8500 3100 50  0001 C CNN
 F 3 "~" V 8500 3100 50  0001 C CNN
 	1    8500 3100
@@
 F 0 "D?" V 9196 3032 50  0000 R CNN
 F 1 "D_Small" V 9105 3032 50  0000 R CNN
-F 2 "" V 9150 3100 50  0001 C CNN
+F 2 "Diode_SMD:D_SOD-123" V 9150 3100 50  0001 C CNN
 F 3 "~" V 9150 3100 50  0001 C CNN
 	1    9150 3100
@@
 F 0 "D?" V 9846 3032 50  0000 R CNN
 F 1 "D_Small" V 9755 3032 50  0000 R CNN
-F 2 "" V 9800 3100 50  0001 C CNN
+F 2 "Diode_SMD:D_SOD-123" V 9800 3100 50  0001 C CNN
 F 3 "~" V 9800 3100 50  0001 C CNN
 	1    9800 3100
@@
 F 0 "D?" V 6596 3682 50  0000 R CNN
 F 1 "D_Small" V 6505 3682 50  0000 R CNN
-F 2 "" V 6550 3750 50  0001 C CNN
+F 2 "Diode_SMD:D_SOD-123" V 6550 3750 50  0001 C CNN
 F 3 "~" V 6550 3750 50  0001 C CNN
 	1    6550 3750
@@
 F 0 "D?" V 7246 3682 50  0000 R CNN
 F 1 "D_Small" V 7155 3682 50  0000 R CNN
-F 2 "" V 7200 3750 50  0001 C CNN
+F 2 "Diode_SMD:D_SOD-123" V 7200 3750 50  0001 C CNN
 F 3 "~" V 7200 3750 50  0001 C CNN
 	1    7200 3750
@@
 F 0 "D?" V 7896 3682 50  0000 R CNN
 F 1 "D_Small" V 7805 3682 50  0000 R CNN
-F 2 "" V 7850 3750 50  0001 C CNN
+F 2 "Diode_SMD:D_SOD-123" V 7850 3750 50  0001 C CNN
 F 3 "~" V 7850 3750 50  0001 C CNN
 	1    7850 3750
@@
 F 0 "D?" V 8546 3682 50  0000 R CNN
 F 1 "D_Small" V 8455 3682 50  0000 R CNN
-F 2 "" V 8500 3750 50  0001 C CNN
+F 2 "Diode_SMD:D_SOD-123" V 8500 3750 50  0001 C CNN
 F 3 "~" V 8500 3750 50  0001 C CNN
 	1    8500 3750
@@
 F 0 "D?" V 9196 3682 50  0000 R CNN
 F 1 "D_Small" V 9105 3682 50  0000 R CNN
-F 2 "" V 9150 3750 50  0001 C CNN
+F 2 "Diode_SMD:D_SOD-123" V 9150 3750 50  0001 C CNN
 F 3 "~" V 9150 3750 50  0001 C CNN
 	1    9150 3750
@@
 F 0 "D?" V 9846 3682 50  0000 R CNN
 F 1 "D_Small" V 9755 3682 50  0000 R CNN
-F 2 "" V 9800 3750 50  0001 C CNN
+F 2 "Diode_SMD:D_SOD-123" V 9800 3750 50  0001 C CNN
 F 3 "~" V 9800 3750 50  0001 C CNN
 	1    9800 3750
@@
 F 0 "D?" V 6596 4332 50  0000 R CNN
 F 1 "D_Small" V 6505 4332 50  0000 R CNN
-F 2 "" V 6550 4400 50  0001 C CNN
+F 2 "Diode_SMD:D_SOD-123" V 6550 4400 50  0001 C CNN
 F 3 "~" V 6550 4400 50  0001 C CNN
 	1    6550 4400
@@
 F 0 "D?" V 7246 4332 50  0000 R CNN
 F 1 "D_Small" V 7155 4332 50  0000 R CNN
-F 2 "" V 7200 4400 50  0001 C CNN
+F 2 "Diode_SMD:D_SOD-123" V 7200 4400 50  0001 C CNN
 F 3 "~" V 7200 4400 50  0001 C CNN
 	1    7200 4400
@@
 F 0 "D?" V 7896 4332 50  0000 R CNN
 F 1 "D_Small" V 7805 4332 50  0000 R CNN
-F 2 "" V 7850 4400 50  0001 C CNN
+F 2 "Diode_SMD:D_SOD-123" V 7850 4400 50  0001 C CNN
 F 3 "~" V 7850 4400 50  0001 C CNN
 	1    7850 4400
@@
 F 0 "D?" V 8546 4332 50  0000 R CNN
 F 1 "D_Small" V 8455 4332 50  0000 R CNN
-F 2 "" V 8500 4400 50  0001 C CNN
+F 2 "Diode_SMD:D_SOD-123" V 8500 4400 50  0001 C CNN
 F 3 "~" V 8500 4400 50  0001 C CNN
 	1    8500 4400
@@
 F 0 "D?" V 9196 4332 50  0000 R CNN
 F 1 "D_Small" V 9105 4332 50  0000 R CNN
-F 2 "" V 9150 4400 50  0001 C CNN
+F 2 "Diode_SMD:D_SOD-123" V 9150 4400 50  0001 C CNN
 F 3 "~" V 9150 4400 50  0001 C CNN
 	1    9150 4400
@@
 F 0 "D?" V 9846 4332 50  0000 R CNN
 F 1 "D_Small" V 9755 4332 50  0000 R CNN
-F 2 "" V 9800 4400 50  0001 C CNN
+F 2 "Diode_SMD:D_SOD-123" V 9800 4400 50  0001 C CNN
 F 3 "~" V 9800 4400 50  0001 C CNN
 	1    9800 4400
@@
 F 0 "D?" V 6596 4982 50  0000 R CNN
 F 1 "D_Small" V 6505 4982 50  0000 R CNN
-F 2 "" V 6550 5050 50  0001 C CNN
+F 2 "Diode_SMD:D_SOD-123" V 6550 5050 50  0001 C CNN
 F 3 "~" V 6550 5050 50  0001 C CNN
 	1    6550 5050
@@
 F 0 "D?" V 7246 4982 50  0000 R CNN
 F 1 "D_Small" V 7155 4982 50  0000 R CNN
-F 2 "" V 7200 5050 50  0001 C CNN
+F 2 "Diode_SMD:D_SOD-123" V 7200 5050 50  0001 C CNN
 F 3 "~" V 7200 5050 50  0001 C CNN
 	1    7200 5050
@@
 F 0 "D?" V 7896 4982 50  0000 R CNN
 F 1 "D_Small" V 7805 4982 50  0000 R CNN
-F 2 "" V 7850 5050 50  0001 C CNN
+F 2 "Diode_SMD:D_SOD-123" V 7850 5050 50  0001 C CNN
 F 3 "~" V 7850 5050 50  0001 C CNN
 	1    7850 5050
@@
 F 0 "D?" V 8546 4982 50  0000 R CNN
 F 1 "D_Small" V 8455 4982 50  0000 R CNN
-F 2 "" V 8500 5050 50  0001 C CNN
+F 2 "Diode_SMD:D_SOD-123" V 8500 5050 50  0001 C CNN
 F 3 "~" V 8500 5050 50  0001 C CNN
 	1    8500 5050
@@
 F 0 "D?" V 9196 4982 50  0000 R CNN
 F 1 "D_Small" V 9105 4982 50  0000 R CNN
-F 2 "" V 9150 5050 50  0001 C CNN
+F 2 "Diode_SMD:D_SOD-123" V 9150 5050 50  0001 C CNN
 F 3 "~" V 9150 5050 50  0001 C CNN
 	1    9150 5050
@@
 F 0 "D?" V 9846 4982 50  0000 R CNN
 F 1 "D_Small" V 9755 4982 50  0000 R CNN
-F 2 "" V 9800 5050 50  0001 C CNN
+F 2 "Diode_SMD:D_SOD-123" V 9800 5050 50  0001 C CNN
 F 3 "~" V 9800 5050 50  0001 C CNN
 	1    9800 5050
@@
 F 0 "D?" V 6596 5632 50  0000 R CNN
 F 1 "D_Small" V 6505 5632 50  0000 R CNN
-F 2 "" V 6550 5700 50  0001 C CNN
+F 2 "Diode_SMD:D_SOD-123" V 6550 5700 50  0001 C CNN
 F 3 "~" V 6550 5700 50  0001 C CNN
 	1    6550 5700
@@
 F 0 "D?" V 7246 5632 50  0000 R CNN
 F 1 "D_Small" V 7155 5632 50  0000 R CNN
-F 2 "" V 7200 5700 50  0001 C CNN
+F 2 "Diode_SMD:D_SOD-123" V 7200 5700 50  0001 C CNN
 F 3 "~" V 7200 5700 50  0001 C CNN
 	1    7200 5700
@@
 F 0 "D?" V 7896 5632 50  0000 R CNN
 F 1 "D_Small" V 7805 5632 50  0000 R CNN
-F 2 "" V 7850 5700 50  0001 C CNN
+F 2 "Diode_SMD:D_SOD-123" V 7850 5700 50  0001 C CNN
 F 3 "~" V 7850 5700 50  0001 C CNN
 	1    7850 5700
@@
 F 0 "D?" V 8546 5632 50  0000 R CNN
 F 1 "D_Small" V 8455 5632 50  0000 R CNN
-F 2 "" V 8500 5700 50  0001 C CNN
+F 2 "Diode_SMD:D_SOD-123" V 8500 5700 50  0001 C CNN
 F 3 "~" V 8500 5700 50  0001 C CNN
 	1    8500 5700
@@
 F 0 "D?" V 9196 5632 50  0000 R CNN
 F 1 "D_Small" V 9105 5632 50  0000 R CNN
-F 2 "" V 9150 5700 50  0001 C CNN
+F 2 "Diode_SMD:D_SOD-123" V 9150 5700 50  0001 C CNN
 F 3 "~" V 9150 5700 50  0001 C CNN
 	1    9150 5700
@@
 F 0 "D?" V 9846 5632 50  0000 R CNN
 F 1 "D_Small" V 9755 5632 50  0000 R CNN
-F 2 "" V 9800 5700 50  0001 C CNN
+F 2 "Diode_SMD:D_SOD-123" V 9800 5700 50  0001 C CNN
 F 3 "~" V 9800 5700 50  0001 C CNN
 	1    9800 5700
@@
 F 0 "D?" V 10496 4982 50  0000 R CNN
 F 1 "D_Small" V 10405 4982 50  0000 R CNN
-F 2 "" V 10450 5050 50  0001 C CNN
+F 2 "Diode_SMD:D_SOD-123" V 10450 5050 50  0001 C CNN
 F 3 "~" V 10450 5050 50  0001 C CNN
 	1    10450 5050
@@
 F 0 "D?" V 10496 5632 50  0000 R CNN
 F 1 "D_Small" V 10405 5632 50  0000 R CNN
-F 2 "" V 10450 5700 50  0001 C CNN
+F 2 "Diode_SMD:D_SOD-123" V 10450 5700 50  0001 C CNN
 F 3 "~" V 10450 5700 50  0001 C CNN
 	1    10450 5700
@@
 F 0 "J?" H 3570 2825 50  0000 C CNN
 F 1 "Conn_01x06" H 3570 2916 50  0000 C CNN
-F 2 "" H 3650 3350 50  0001 C CNN
+F 2 "Connector_PinSocket_2.54mm:PinSocket_1x06_P2.54mm_Vertical" H 3650 3350 50  0001 C CNN
 F 3 "~" H 3650 3350 50  0001 C CNN
 	1    3650 3350

Commit message: add more annotation
Parts:
- added C? (x2): C_Small, Capacitor_SMD:C_0603_1608Metric_Pad1.05x0.95mm_HandSolder, symbol Device:C_Small
- added R? (x2): R_Small, Resistor_SMD:R_0603_1608Metric_Pad1.05x0.95mm_HandSolder, symbol Device:R_Small
- added Y?: Crystal_GND24_Small, symbol Device:Crystal_GND24_Small
- C? (x4): footprint (none) -> Capacitor_SMD:C_0603_1608Metric_Pad1.05x0.95mm_HandSolder
- R?: footprint (none) -> Resistor_SMD:R_0603_1608Metric_Pad1.05x0.95mm_HandSolder
- gave numbers to parts that had none: 67
Connections:
- net GND: now also C?.1, C?.1, Y?.2, Y?.4
- net OSC_IN: now also C?.2, Y?.1
- net OSC_OUT: now also C?.2, Y?.3
- net VDD: now also R?.1, R?.1
- net at J2.R1: now also R?.2
- net at J2.R2: now also R?.2
