File: RNA.kicad_pcb (KiCad board)
At the start: 2 copper layers, 134 x 177 mm, 164 parts, among them J1 USB_B_Micro, J2 SM04B-SRSS-TB(LF)(SN), J3 AudioJack4, J4 Conn_01x06, J5 SM04B-SRSS-TB(LF)(SN), SW1 SW_SPST, SW10 CPG135001S30, SW11 CPG135001S30, SW12 CPG135001S30, SW13 CPG135001S30, SW14 CPG135001S30, SW15 CPG135001S30, SW16 CPG135001S30, SW17 CPG135001S30, SW18 CPG135001S30, SW19 CPG135001S30, SW2 SW_Push, SW20 CPG135001S30, SW21 CPG135001S30, SW22 CPG135001S30, SW23 CPG135001S30, SW24 CPG135001S30, SW25 CPG135001S30, SW26 CPG135001S30, SW27 CPG135001S30, SW28 CPG135001S30, SW29 CPG135001S30, SW3 CPG135001S30, SW30 CPG135001S30, SW31 CPG135001S30, SW32 CPG135001S30, SW33 CPG135001S30, SW34 CPG135001S30, SW35 CPG135001S30, SW36 CPG135001S30, SW37 CPG135001S30, SW38 CPG135001S30, SW39 CPG135001S30, SW4 CPG135001S30, SW40 CPG135001S30, SW41 CPG135001S30, SW42 CPG135001S30, SW43 CPG135001S30, SW44 CPG135001S30, SW45 CPG135001S30, SW46 CPG135001S30, SW47 CPG135001S30, SW48 CPG135001S30, SW49 CPG135001S30, SW5 CPG135001S30, SW50 CPG135001S30, SW51 CPG135001S30, SW52 CPG135001S30, SW53 CPG135001S30, SW54 CPG135001S30, SW55 CPG135001S30, SW56 CPG135001S30, SW57 CPG135001S30, SW58 CPG135001S30, SW59 CPG135001S30, SW6 CPG135001S30, SW60 CPG135001S30, SW61 CPG135001S30, SW62 CPG135001S30, SW63 CPG135001S30, SW64 CPG135001S30, SW65 CPG135001S30, SW66 CPG135001S30, SW7 CPG135001S30, SW8 CPG135001S30, SW9 CPG135001S30, U1 STM32F072C8Tx, U2 PRTR5V0U2X, U3 MCP1703A-3302_SOT23, U4 CAT24M01W, U5 MCP23017_SS

Commit message: more routing
Parts:
- added REF**: MountingHole_2.2mm_M2_Pad_Via, MountingHole:MountingHole_2.2mm_M2_Pad_Via, F.Cu at (74.0, 71.0)
- C1, C2, C3, C4, C5: footprint Capacitor_SMD:C_0603_1608Metric -> Capacitor_SMD:C_0402_1005Metric
- U4: value CAT24M01W -> CAT250xxx
- moved U4 43.8 mm to (128.8, 30.8), turned to 270 degrees
- moved C8 39.6 mm to (125.1, 31.1)
- moved SW1 5.08 mm to (141.2, 61.7), turned to 0 degrees
- moved R1 2.59 mm to (138.6, 47.5)
- moved C7 1.62 mm to (143.5, 35.1), turned to 0 degrees
- moved SW2 1.54 mm to (144.7, 68.0)
- moved C5 1.22 mm to (136.9, 46.9), turned to 270 degrees
- moved C2 0.39 mm to (138.9, 33.8)
- moved C1 0.36 mm to (142.7, 42.7)
- moved C3 0.21 mm to (135.4, 46.5)
- moved C4 0.11 mm to (130.1, 37.7)
Connections:
- J2 pad 2: SCL3 -> SCL2
- J2 pad 3: SDA3 -> SDA2
- R2 pad 2: SDA3 -> SDA2
- R3 pad 2: SCL3 -> SCL2
- U1 pad 15: Net-(U1-Pad15) -> SCK
- U1 pad 16: Net-(U1-Pad16) -> MISO
- U1 pad 17: SCL3 -> MOSI
- U1 pad 26: COL6 -> SCL2
- U1 pad 27: COL7 -> SDA2
- U1 pad 40: SDA3 -> COL6
- U1 pad 41: Net-(U1-Pad41) -> COL7
- U4 pad 1: Net-(U4-Pad1) -> GND
- U4 pad 2: GND -> MISO
- U4 pad 3: GND -> VDD
- U4 pad 5: SDA1 -> MOSI
- U4 pad 6: SCL1 -> SCK
- U4 pad 7: GND -> VDD
Routing:
- net COL7S: track 222.7 -> 0.00 mm
- net COL6S: track 210.1 -> 0.00 mm
- net COL5S: track 178.8 -> 0.00 mm
- net ROW1S: track 174.3 -> 0.00 mm, vias 6 -> 0
- net ROW5S: track 164.1 -> 0.00 mm
- net COL4S: track 158.7 -> 0.00 mm
- net GND: track 236.1 -> 77.8 mm, vias 16 -> 6
- net ROW4S: track 150.0 -> 0.00 mm, vias 7 -> 0
- net ROW2S: track 149.3 -> 0.00 mm, vias 6 -> 0
- net ROW4: track 192.8 -> 46.9 mm, vias 2 -> 0
- net COL1: track 242.6 -> 102.0 mm
- net ROW3S: track 134.7 -> 0.00 mm, vias 6 -> 0
- net COL3S: track 132.6 -> 0.00 mm
- net COL2: track 215.7 -> 93.0 mm, vias 4 -> 2
- net COL2S: track 111.6 -> 0.00 mm, vias 3 -> 0
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